File: hardware/remote_control.sch (EAGLE design)
At the start: 52 parts, among them IC1 MCP4726, IC3 REG1117, IC4 TL072D, IC5 LM4041A12DBZ

Commit message: rfsw
Parts:
- removed C11, C12: (no value), resistor:C-EUC0805
- removed D9: TS4148, jason_eagle6:TS4148
- removed FB1: (no value), microbuilder:FERRITE
- removed JP1: (no value), pinhead:PINHD-1X3
- removed R16: (no value), rcl:R-EU_R0805
- removed S1: (no value), switch-omron:10-XX
- removed U$1: PIC16F1825SO14, jasons_stuff:PIC16F1825SO14
- removed U$10, U$8, U$9: MICRO-SPDT, jason_eagle6:MICRO-SPDT
- removed U$6: SN74LVC2G14, jason_eagle6:SN74LVC2G14
- added C3: (no value), resistor:C-EUC0805
- added D2: TS4148, jason_eagle6:TS4148
- added IC2: PIC16F1825SO14, jasons_stuff:PIC16F1825SO14
- added IC6: SN74LVC2G14, jason_eagle6:SN74LVC2G14
- added IR_DET: (no value), pinhead:PINHD-1X3
- added L1: (no value), microbuilder:FERRITE
- added R2, R3: (no value), rcl:R-EU_R0805
- added SW1: (no value), switch-omron:10-XX
- added SW2, SW3, SW4: MICRO-SPDT, jason_eagle6:MICRO-SPDT
- C10, C9: device resistor:C-EUC0805 -> resistor:CPOL-EUE2-5
- C2, C4: device resistor:CPOL-EUE2-5 -> resistor:C-EUC0805
- IC1: value MCP4726 -> REG1117; device jasons_stuff:MCP4726 -> burr-brown:REG1117
- IC3: value REG1117 -> LM4041A12DBZ; device burr-brown:REG1117 -> texas:LM4041A12DBZ
- IC4: value TL072D -> MCP4726; device linear:TL072D -> jasons_stuff:MCP4726
- IC5: value LM4041A12DBZ -> TL072D; device texas:LM4041A12DBZ -> linear:TL072D
- R1: value (none) -> 3k
- R14: value 3k -> (none)
- R8: device rcl:R-EU_R0805 -> resistor:C-EUC0805
Connections:
- net +12V: now also C1.2, C6.1, C9.+, IC1.VIN, IC5P.V+, L1.P$2; no longer C12.1, C4.+, C5.2, FB1.P$2, IC3.VIN, IC4P.V+
- net CLOCK_IN: now also IC2.RC5/RX, IC6.1Y; no longer U$1.RC5/RX, U$6.1Y
- net CV_OUT: now also IC4.VOUT, IC5A.+IN; no longer IC1.VOUT, IC4A.+IN
- net GATE_OUT: now also IC2.RC2, IC5B.+IN; no longer IC4B.+IN, U$1.RC2
- net GND: now also C10.-, C2.1, C3.1, C4.1, C5.2, C6.2, C7.1, C9.-, D6.A, D8.A, IC1.GND, IC2.VSS, IC3.A, IC4.VSS, IC5P.V-, IC6.GND, IR_DET.2, R10.2, R12.2, R4.2, R6.2, SW1.P, SW1.P1; no longer C10.1, C12.2, C2.-, C4.-, C5.1, C6.1, C7.2, C9.1, D3.A, D5.A, IC1.VSS, IC3.GND, IC4P.V-, IC5.A, JP1.2, R13.2, R5.2, R7.2, R9.2, S1.P, S1.P1, U$1.VSS, U$6.GND
- net IR_RX: now also IC2.RA2/INT, IR_DET.1; no longer JP1.1, U$1.RA2/INT
- net N$10: now also R11.1; no longer R4.1
- net N$11: now also D2.A, SW4.COM; no longer D7.A, U$8.COM
- net N$13: now also IC5B.OUT, R14.1, R15.2, R5.1; no longer IC4B.OUT, R1.1, R10.1, R8.2
- net N$14: now also D7.A, D8.C, IC6.1A, R12.1, R13.2; no longer D5.C, D6.A, R6.2, R7.1, U$6.1A
- net N$15: now also D3.A, SW3.COM; no longer D8.A, U$9.COM
- net N$16: now also C8.2, R15.1; no longer C10.2, R8.1
- net N$17: now also IC5B.-IN, R4.1, R5.2; no longer IC4B.-IN, R10.2, R9.1
- net N$18: now also IC5A.-IN, R6.1, R7.2, R8.1; no longer C11.1, IC4A.-IN, R12.2, R13.1
- net N$19: now also R7.1, R9.1; no longer R11.1, R12.1
- net N$2: now also IC2.RA3/MCLR#/VPP, SW1.S, SW1.S1; no longer S1.S, S1.S1, U$1.RA3/MCLR#/VPP
- net N$20: now also IC5A.OUT, R8.2, R9.2; no longer C11.2, IC4A.OUT, R11.2
- net N$25: now also D4.A, SW2.COM; no longer D9.A, U$10.COM
- net N$4: now also L1.P$1; no longer FB1.P$1
- net N$5: now also R14.2; no longer R1.2
- net N$6: now also C4.2, IC3.C, IC4.VREF, R1.1; no longer C9.2, IC1.VREF, IC5.C, R14.1
- net N$9: now also R13.1; no longer R6.1
- net READ1: now also IC2.RC4/TX, SW2.A, SW3.A, SW4.A; no longer U$1.RC4/TX, U$10.A, U$8.A, U$9.A
- net READ2: now also IC2.RC3/SS#, SW2.B, SW3.B, SW4.B; no longer U$1.RC3/SS#, U$10.B, U$8.B, U$9.B
- net SCAN1: now also D2.C, IC2.RA0/ICSPDAT; no longer D7.C, U$1.RA0/ICSPDAT
- net SCAN2: now also D3.C, IC2.RA1/ICPCLK; no longer D8.C, U$1.RA1/ICPCLK
- net SCAN3: now also D4.C, IC2.RA4/SDO; no longer D9.C, U$1.RA4/SDO
- net SCL: now also IC2.RCO/SCL/SCK, IC4.SCL, R3.1; no longer IC1.SCL, R15.1, U$1.RCO/SCL/SCK
- net SDA: now also IC2.RC1/SDA/SDI, IC4.SDA, R2.1; no longer IC1.SDA, R16.1, U$1.RC1/SDA/SDI
- net TRIG_IN: now also IC2.RA5, IC6.2Y; no longer U$1.RA5, U$6.2Y
- net VDD: now also C10.+, C2.2, C3.2, C5.1, C7.2, D5.C, D7.C, IC1.VOUT, IC2.VDD, IC4.VDD, IC6.VCC, IR_DET.3, R1.2, R2.2, R3.2; no longer C1.2, C2.+, C6.2, C7.1, C8.2, D4.C, D6.C, IC1.VDD, IC3.VOUT, JP1.3, R14.2, R15.2, R16.2, U$1.VDD, U$6.VCC
- net X: now also D5.A, D6.C, IC6.2A, R10.1, R11.2; no longer D3.C, D4.A, R4.2, R5.1, U$6.2A
Other:
- note added: "2020/Sixty-Four Pixels Ltd"
- note added: "CC-BY-NC-SA"
- note added: "CV Out Buffer"
- note added: "Detector"
- note added: "Gate Out Buffer"
- note added: "IRL - INFRA RED LISTENER rev 1"
- note added: "Input Buffer / Schmitt Trigger"
- note added: "PIC16F1825"
- note added: "Power Supply"
- note added: "Switches ON-OFF-ON"
- moved on the sheet: C1, C5, C6, C7, C8, CLOCK_IN, CV_OUT, D1, D3, D4, D5, D6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

Commit message: ww
Other:
- note added: "***DO NOT USE TL072 - USE SINGLE SUPPLY OPAMP LM358 OR BETTER ***"
Changed lines of the file:
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@@
 <text x="17.018" y="-3.81" size="4.572" layer="91">2020/Sixty-Four Pixels Ltd </text>
 <text x="17.018" y="-11.43" size="4.572" layer="91">CC-BY-NC-SA</text>
+<text x="349.758" y="58.674" size="3.81" layer="91">***DO NOT USE TL072 - USE SINGLE SUPPLY OPAMP LM358 OR BETTER ***</text>
 </plain>
 <instances>

Commit message: sdf
Connections:
- net GND: now also IR_DET.3; no longer IR_DET.2
- net VDD: now also IR_DET.2; no longer IR_DET.3
Changed lines of the file:
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@@
 </segment>
 <segment>
-<pinref part="IR_DET" gate="A" pin="2"/>
-<wire x1="218.44" y1="30.48" x2="226.06" y2="30.48" width="0.1524" layer="91"/>
 <pinref part="GND25" gate="1" pin="GND"/>
 <wire x1="226.06" y1="25.4" x2="226.06" y2="30.48" width="0.1524" layer="91"/>
+<pinref part="IR_DET" gate="A" pin="3"/>
+<wire x1="218.44" y1="33.02" x2="226.06" y2="30.48" width="0.1524" layer="91"/>
 </segment>
 <segment>
@@
 <net name="VDD" class="0">
 <segment>
-<pinref part="IR_DET" gate="A" pin="3"/>
-<wire x1="218.44" y1="33.02" x2="226.06" y2="33.02" width="0.1524" layer="91"/>
 <pinref part="U$14" gate="G$1" pin="VDD"/>
 <wire x1="226.06" y1="38.1" x2="226.06" y2="33.02" width="0.1524" layer="91"/>
-</segment>
-<segment>
+<pinref part="IR_DET" gate="A" pin="2"/>
+<wire x1="218.44" y1="30.48" x2="226.06" y2="33.02" width="0.1524" layer="91"/>
+</segment>
+<segment>

Commit message: board updates
Parts:
- removed CLOCK_IN: WQP-PJ301M-12_JACK, thonkiconn:WQP-PJ301M-12_JACK
- removed D7, D8: TS4148, jason_eagle6:TS4148
- removed IC6: SN74LVC2G14, jason_eagle6:SN74LVC2G14
- removed R15: (no value), rcl:R-EU_R0805
- added CLK_IN: THONKICONN_STEREO, jason_eagle6:THONKICONN_STEREO
- added Q1, Q2: (no value), transistor-neu-to92:MMBT3904LT1-NPN-SOT23-BEC
- R8: device resistor:C-EUC0805 -> rcl:R-EU_R0805
- renumbered J1 to ICSP
Connections:
- removed net N$14: D7.A, D8.C, IC6.1A, R12.1, R13.2
- removed net X: D5.A, D6.C, IC6.2A, R10.1, R11.2
- new net N$12: D5.C, R9.2
- new net N$21: Q1.B, R9.1
- new net N$3: CLK_IN.T, D6.A
- new net N$7: D6.C, R10.2
- net CLOCK_IN: now also Q2.E, R13.1; no longer IC6.1Y
- net GND: now also CLK_IN.S, R13.2; no longer C7.1, CLOCK_IN.1, D6.A, D8.A, IC6.GND, R10.2
- net N$10: now also D5.A; no longer R11.1
- net N$13: now also R11.1, R14.2; no longer R14.1, R15.2
- net N$16: now also R14.1; no longer R15.1
- net N$18: now also C7.1; no longer R8.1
- net N$19: now also R8.1; no longer R9.1
- net N$20: now also C7.2; no longer R9.2
- net N$5: now also R11.2; no longer R14.2
- net N$9: now also Q2.B, R10.1; no longer CLOCK_IN.2, R13.1
- net TRIG_IN: now also Q1.E, R12.1; no longer IC6.2Y
- net VDD: now also Q1.C, Q2.C; no longer C7.2, D5.C, D7.C, IC6.VCC
Other:
- note added: "2021/Sixty-Four Pixels Ltd"
- note added: "CLOCK/MIDI IN BUFFER"
- note added: "CV.TV - IR SEQUENCER rev 2"
- note added: "TRIG IN BUFFER"
- note removed: "2020/Sixty-Four Pixels Ltd"
- note removed: "IRL - INFRA RED LISTENER rev 1"
- note removed: "Input Buffer / Schmitt Trigger"
- moved on the sheet: C3, C7, D5, D6, R10, R11, R12, R13, R14, R8, R9, TRIG_IN
