File: hardware/cvtv.brd (EAGLE design)
At the start: 19.6 x 100.1 mm, 50 parts, among them IC1 REG1117, IC2 PIC16F1825SO14, IC3 LM4041A12DBZ, IC4 MCP4726, IC5 TL072D, SW2 MICRO-SPDT, SW3 MICRO-SPDT, SW4 MICRO-SPDT

Commit message: check in updates
Parts:
- C6: value (none) -> 100n
- C7: value (none) -> 20p
- C8: value (none) -> 10n
- R10, R14, R8, R9: value (none) -> 1k
- R11, R12, R13, R2, R3: value (none) -> 4k7
- R4, R5, R6, R7: value (none) -> 10k
